Commit message: Fix broken arm and floating imu_link in Gazebo SDF
Two bugs fixed:
1. Restore explicit <pose> on all arm links (arm_base_link..arm_link_6):
   SDF requires absolute poses in the model frame to set initial joint
   configuration. Without them all links default to origin and the arm
   collapses on spawn.

2. Add imu_joint (base_link → imu_link at -0.032 0 0.068) and explicit
   pose on imu_link: the link was defined with no joint, causing it to
   appear as a floating unattached piece in Gazebo.

Co-Authored-By: Claude Sonnet 4.6 <noreply@anthropic.com>

File: ros2_ws/src/tb3_description/urdf/gz_waffle_arm.sdf.xacro (robot description, xacro)
@@ -54,4 +54,5 @@
       </link>
       <link name="imu_link">
+        <pose>-0.032 0 0.078 0 0 0</pose>
         <sensor name="tb3_imu" type="imu">
           <always_on>true</always_on>
@@ -313,4 +314,9 @@
         <axis><xyz>0 0 1</xyz></axis>
       </joint>
+      <joint name="imu_joint" type="fixed">
+        <parent>base_link</parent>
+        <child>imu_link</child>
+        <pose>-0.032 0 0.068 0 0 0</pose>
+      </joint>
       <!-- ================================================================ -->
       <!-- IRB120 ARM LINKS (prefix: arm_)                                   -->
@@ -318,4 +324,5 @@
       <!-- ================================================================ -->
       <link name="arm_base_link">
+        <pose>0 0 0.10 0 0 0</pose>
         <gravity>false</gravity>
         <inertial>
@@ -344,4 +351,5 @@
       </link>
       <link name="arm_link_1">
+        <pose>0 0 0.10 0 0 0</pose>
         <gravity>false</gravity>
         <inertial>
@@ -366,4 +374,5 @@
       </link>
       <link name="arm_link_2">
+        <pose>0 0 0.39 0 0 0</pose>
         <gravity>false</gravity>
         <inertial>
@@ -388,4 +397,5 @@
       </link>
       <link name="arm_link_3">
+        <pose>0 0 0.66 0 0 0</pose>
         <gravity>false</gravity>
         <inertial>
@@ -410,4 +420,5 @@
       </link>
       <link name="arm_link_4">
+        <pose>0 0 0.73 0 0 0</pose>
         <gravity>false</gravity>
         <inertial>
@@ -432,4 +443,5 @@
       </link>
       <link name="arm_link_5">
+        <pose>0.302 0 0.73 0 0 0</pose>
         <gravity>false</gravity>
         <inertial>
@@ -454,4 +466,5 @@
       </link>
       <link name="arm_link_6">
+        <pose>0.374 0 0.73 0 0 0</pose>
         <gravity>false</gravity>
         <inertial>
